File: pcb/banime40/banime40.kicad_sch (KiCad schematic)
At the start: 88 parts, among them SW1 SW_SPST, SW10 SW_SPST, SW11 SW_SPST, SW12 SW_SPST, SW13 SW_SPST, SW14 SW_SPST, SW15 SW_SPST, SW16 SW_SPST, SW17 SW_SPST, SW18 SW_SPST, SW19 SW_SPST, SW2 SW_SPST, SW20 SW_SPST, SW21 SW_SPST, SW22 SW_SPST, SW23 SW_SPST, SW24 SW_SPST, SW25 SW_SPST, SW26 SW_SPST, SW27 SW_SPST, SW28 SW_SPST, SW29 SW_SPST, SW3 SW_SPST, SW30 SW_SPST, SW31 SW_SPST, SW32 SW_SPST, SW33 SW_SPST, SW34 SW_SPST, SW35 SW_SPST, SW36 SW_SPST, SW37 SW_SPST, SW38 SW_SPST, SW39 SW_SPST, SW4 SW_SPST, SW40 SW_SPST, SW41 SW_SPST, SW42 SW_SPST, SW43 SW_SPST, SW44 SW_SPST, SW45 SW_SPST, SW47 RotaryEncoder_Switch, SW5 SW_SPST, SW6 SW_SPST, SW7 SW_SPST, SW8 SW_SPST, SW9 SW_SPST, U1 ProMicro

Commit message: create patch fix for rotary encoders
Parts:
- SW46: value (none) -> RotaryEncoder_Switch; footprint (none) -> Keebio-Parts:RotaryEncoder_EC11
- SW47: footprint (none) -> Keebio-Parts:RotaryEncoder_EC11
Connections:
- net gnd: now also SW44.1 (A), SW45.1 (A), U1.23 (GND); no longer SW44.2 (B), SW45.2 (B), U1.22 (RST)
- new net: SW44.2 (B), SW45.2 (B)
Changed lines of the file:
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@@
   (junction (at 95.25 33.02) (diameter 0) (color 0 0 0 0)
   )
-  (junction (at 74.93 30.48) (diameter 0) (color 0 0 0 0)
-  )
   (junction (at 161.29 40.64) (diameter 0) (color 0 0 0 0)
   )
@@
   )
   (junction (at 146.05 82.55) (diameter 0) (color 0 0 0 0)
-  )
-  (junction (at 73.66 33.02) (diameter 0) (color 0 0 0 0)
   )
   (junction (at 85.09 40.64) (diameter 0) (color 0 0 0 0)
@@
     (stroke (width 0) (type default) (color 0 0 0 0))
   )
-  (wire (pts (xy 73.66 33.02) (xy 74.93 33.02))
-    (stroke (width 0) (type default) (color 0 0 0 0))
-  )
   (wire (pts (xy 100.33 73.66) (xy 115.57 73.66))
     (stroke (width 0) (type default) (color 0 0 0 0))
@@
   )
   (wire (pts (xy 110.49 49.53) (xy 110.49 66.04))
-    (stroke (width 0) (type default) (color 0 0 0 0))
-  )
-  (wire (pts (xy 74.93 33.02) (xy 74.93 30.48))
     (stroke (width 0) (type default) (color 0 0 0 0))
   )
@@
     )
   )
-  (global_label "gnd" (shape input) (at 74.93 33.02 0) (fields_autoplaced)
+  (global_label "gnd" (shape input) (at 62.23 30.48 90) (fields_autoplaced)
     (effects (font (size 1.27 1.27)) (justify left))
-    (property "Intersheet References" "${INTERSHEET_REFS}" (id 0) (at 80.7013 32.9406 0)
+    (property "Intersheet References" "${INTERSHEET_REFS}" (id 0) (at 62.1506 24.7087 90)
       (effects (font (size 1.27 1.27)) (justify left) hide)
     )
@@
       (effects (font (size 1.27 1.27)) (justify right))
     )
-    (property "Footprint" "" (id 2) (at 223.266 96.52 0)
+    (property "Footprint" "Keebio-Parts:RotaryEncoder_EC11" (id 2) (at 223.266 96.52 0)
       (effects (font (size 1.27 1.27)) hide)
     )
@@
       (effects (font (size 1.27 1.27)) (justify right))
     )
-    (property "Value" "" (id 1) (at 96.012 94.4122 90)
+    (property "Value" "RotaryEncoder_Switch" (id 1) (at 96.012 94.4122 90)
       (effects (font (size 1.27 1.27)) (justify right))
     )
-    (property "Footprint" "" (id 2) (at 86.106 96.52 0)
-      (effects (font (size 1.27 1.27)) hide)
-    )
+    (property "Footprint" "Keebio-Parts:RotaryEncoder_EC11" (id 2) (at 86.106 96.52 0)
+      (effects (font (size 1.27 1.27)) hide)
+    )
